File: ncv7240-driver.kicad_pcb (KiCad board)
At the start: 2 copper layers, 0 parts

Commit message: Start PCB layout: 4-layer 160x100mm with floorplan and pours
- tools/gen_pcb.py — deterministic PCB skeleton generator
- 160 × 100 mm rectangular board outline on Edge.Cuts
- 4-layer stackup: F.Cu / GND (In1) / +24V (In2) / B.Cu, 1.6 mm FR4 ENIG
- 4× M3 mounting holes inset 4 mm from corners
- 57 nets pre-declared (matches schematic: GND/+24V/+3V3/VBUS/CC/I2C/
  SPI/PD/USB/RST_BTN/BOOT_BTN + OUT1..OUT32)
- GND copper pours on In1.Cu and B.Cu; +24V pour on In2.Cu
- Floorplan annotated on User.Comments (USB-C/PD, Buck, ESP32,
  4×NCV7240, screw terminals, flyback diode field)
- F.SilkS header text 'NCV7240 x4 Driver — 24V PD EPR'

Open in KiCad and run 'Tools → Update PCB from Schematic' to pull
in the footprints from the standard KiCad libraries.

README updated with Bürkert 0127 load notes, flyback-diode design
intent (EMI loop near terminals), and ASCII floorplan.
Parts:
- added MH1: M3, MountingHole:MountingHole_3.2mm_M3, F.Cu at (4.00, 4.00)
- added MH2: M3, MountingHole:MountingHole_3.2mm_M3, F.Cu at (156.0, 4.00)
- added MH3: M3, MountingHole:MountingHole_3.2mm_M3, F.Cu at (4.00, 96.0)
- added MH4: M3, MountingHole:MountingHole_3.2mm_M3, F.Cu at (156.0, 96.0)
Routing:
- added copper zone on In2.Cu, net +24V
- added copper zone on B.Cu, net GND
- added copper zone on In1.Cu, net GND
Other:
- board outline added: 160 x 100 mm
- copper layers 2 -> 4
- rule pad_to_mask_clearance: 0 -> 0.05
- board text added: "4× NCV7240 (U3..U6 + decoupling)"
- board text added: "Buck 24V→3V3 (U7, L1, C3, R6/R7)"
- board text added: "ESP32-S3 (U2, C4/C5, R1..R5)"
- board text added: "Flyback diode field (D2..D33, B260A, K→+24V)"
- board text added: "NCV7240 x4 Driver — 24V PD EPR"
- board text added: "Screw terminals (J2..J5, 32 outputs)"
- board text added: "USB-C PD (J1, U1, C1/C2, D1)"
- board text added: "rev 0.1 — 2026"

Commit message: Pre-place all 72 footprints into floorplan with net assignments
200×120 mm 4-layer board, all components placed with embedded pad
geometry so kicanvas can render the board directly. After opening in
KiCad, 'Tools → Update PCB from Schematic' will refresh footprints
to the full library geometry while preserving placement and nets.

Placement (left → right):
  - USB-C J1 + AP33772S U1 + bulk caps C1/C2 + TVS D1
  - Buck U7 (TPS62932 SOT-23-6) + L1 + C3 + C6 + C7 + R6/R7
  - ESP32-S3 U2 with decoupling C4/C5 + pull-up bank R1..R5
  - 4× NCV7240 (U3..U6) stacked vertically at x=108,
    y={18,46,74,102} with local 100nF + 10uF decoupling per IC
  - 32× B260A SMA flyback diodes (D2..D33) in 2×4 columns
    next to each NCV (cathode→+24V, anode→OUTx)
  - 4× Phoenix MKDS-1,5-8 screw terminals (J2..J5) at x=180

Routing:
  - GND pour on In1.Cu and B.Cu (full board)
  - +24V plane on In2.Cu (full board)
  - +3V3 island on F.Cu top-left around ESP32/buck
  - 48 GND stitching vias around board perimeter
  - All pad nets correctly assigned (313 pads, 62 nets)

Left for the user / KiCad autorouter: 32× OUTx fanout from NCV
to flyback diode to screw terminal (regular pattern, ~5 mm each),
SPI bus and I2C signal traces on F.Cu.
Parts:
- added C1: 100uF/50V, Capacitor_SMD:CP_Elec_10x10.5, F.Cu at (46.0, 24.0)
- added C10: 100nF, Capacitor_SMD:C_0603_1608Metric, F.Cu at (120.0, 13.0)
- added C11: 10uF/50V, Capacitor_SMD:C_1210_3225Metric, F.Cu at (120.0, 23.0)
- added C12: 100nF, Capacitor_SMD:C_0603_1608Metric, F.Cu at (120.0, 41.0)
- added C13: 10uF/50V, Capacitor_SMD:C_1210_3225Metric, F.Cu at (120.0, 51.0)
- added C14: 100nF, Capacitor_SMD:C_0603_1608Metric, F.Cu at (120.0, 69.0)
- added C15: 10uF/50V, Capacitor_SMD:C_1210_3225Metric, F.Cu at (120.0, 79.0)
- added C16: 100nF, Capacitor_SMD:C_0603_1608Metric, F.Cu at (120.0, 97.0)
- added C17: 10uF/50V, Capacitor_SMD:C_1210_3225Metric, F.Cu at (120.0, 107.0)
- added C2: 10uF/50V, Capacitor_SMD:C_1210_3225Metric, F.Cu at (46.0, 34.0)
- added C3: 22uF, Capacitor_SMD:C_0805_2012Metric, F.Cu at (36.0, 60.0)
- added C4: 10uF, Capacitor_SMD:C_0805_2012Metric, F.Cu at (60.0, 22.0)
- added C5: 100nF, Capacitor_SMD:C_0603_1608Metric, F.Cu at (60.0, 28.0)
- added C6: 100nF, Capacitor_SMD:C_0603_1608Metric, F.Cu at (18.0, 53.0)
- added C7: 100nF, Capacitor_SMD:C_0603_1608Metric, F.Cu at (12.0, 60.0)
- added D1: SMBJ33A, Diode_SMD:D_SMB, F.Cu at (52.0, 30.0)
- added D10: B260A, Diode_SMD:D_SMA, F.Cu at (140.0, 39.5)
- added D11: B260A, Diode_SMD:D_SMA, F.Cu at (140.0, 43.5)
- added D12: B260A, Diode_SMD:D_SMA, F.Cu at (140.0, 47.5)
- added D13: B260A, Diode_SMD:D_SMA, F.Cu at (140.0, 51.5)
- added D14: B260A, Diode_SMD:D_SMA, F.Cu at (148.0, 39.5)
- added D15: B260A, Diode_SMD:D_SMA, F.Cu at (148.0, 43.5)
- added D16: B260A, Diode_SMD:D_SMA, F.Cu at (148.0, 47.5)
- added D17: B260A, Diode_SMD:D_SMA, F.Cu at (148.0, 51.5)
- added D18: B260A, Diode_SMD:D_SMA, F.Cu at (140.0, 67.5)
- added D19: B260A, Diode_SMD:D_SMA, F.Cu at (140.0, 71.5)
- added D2: B260A, Diode_SMD:D_SMA, F.Cu at (140.0, 11.5)
- added D20: B260A, Diode_SMD:D_SMA, F.Cu at (140.0, 75.5)
- added D21: B260A, Diode_SMD:D_SMA, F.Cu at (140.0, 79.5)
- added D22: B260A, Diode_SMD:D_SMA, F.Cu at (148.0, 67.5)
- added D23: B260A, Diode_SMD:D_SMA, F.Cu at (148.0, 71.5)
- added D24: B260A, Diode_SMD:D_SMA, F.Cu at (148.0, 75.5)
- added D25: B260A, Diode_SMD:D_SMA, F.Cu at (148.0, 79.5)
- added D26: B260A, Diode_SMD:D_SMA, F.Cu at (140.0, 95.5)
- added D27: B260A, Diode_SMD:D_SMA, F.Cu at (140.0, 99.5)
- added D28: B260A, Diode_SMD:D_SMA, F.Cu at (140.0, 103.5)
- added D29: B260A, Diode_SMD:D_SMA, F.Cu at (140.0, 107.5)
- added D3: B260A, Diode_SMD:D_SMA, F.Cu at (140.0, 15.5)
- added D30: B260A, Diode_SMD:D_SMA, F.Cu at (148.0, 95.5)
- added D31: B260A, Diode_SMD:D_SMA, F.Cu at (148.0, 99.5)
- added D32: B260A, Diode_SMD:D_SMA, F.Cu at (148.0, 103.5)
- added D33: B260A, Diode_SMD:D_SMA, F.Cu at (148.0, 107.5)
- added D4: B260A, Diode_SMD:D_SMA, F.Cu at (140.0, 19.5)
- added D5: B260A, Diode_SMD:D_SMA, F.Cu at (140.0, 23.5)
- added D6: B260A, Diode_SMD:D_SMA, F.Cu at (148.0, 11.5)
- added D7: B260A, Diode_SMD:D_SMA, F.Cu at (148.0, 15.5)
- added D8: B260A, Diode_SMD:D_SMA, F.Cu at (148.0, 19.5)
- added D9: B260A, Diode_SMD:D_SMA, F.Cu at (148.0, 23.5)
- added J1: USB-C, Connector:USB_C_Receptacle_HRO_TYPE-C-31-M-12, F.Cu at (12.0, 30.0)
- added J2: OUT1-8, TerminalBlock:TerminalBlock_Phoenix_MKDS-1,5-8_1x08_P5.00mm_Horizontal, F.Cu at (180.0, 18.0)
- added J3: OUT9-16, TerminalBlock:TerminalBlock_Phoenix_MKDS-1,5-8_1x08_P5.00mm_Horizontal, F.Cu at (180.0, 46.0)
- added J4: OUT17-24, TerminalBlock:TerminalBlock_Phoenix_MKDS-1,5-8_1x08_P5.00mm_Horizontal, F.Cu at (180.0, 74.0)
- added J5: OUT25-32, TerminalBlock:TerminalBlock_Phoenix_MKDS-1,5-8_1x08_P5.00mm_Horizontal, F.Cu at (180.0, 102.0)
- added L1: 4.7uH/2A, Inductor_SMD:L_Bourns-SRN6045TA, F.Cu at (28.0, 60.0)
- added R1: 10k, Resistor_SMD:R_0603_1608Metric, F.Cu at (92.0, 16.0)
- added R2: 10k, Resistor_SMD:R_0603_1608Metric, F.Cu at (92.0, 20.0)
- added R3: 10k, Resistor_SMD:R_0603_1608Metric, F.Cu at (92.0, 24.0)
- added R4: 4.7k, Resistor_SMD:R_0603_1608Metric, F.Cu at (92.0, 28.0)
- added R5: 4.7k, Resistor_SMD:R_0603_1608Metric, F.Cu at (92.0, 32.0)
- added R6: 100k, Resistor_SMD:R_0603_1608Metric, F.Cu at (22.0, 70.0)
- added R7: 20k, Resistor_SMD:R_0603_1608Metric, F.Cu at (30.0, 70.0)
- added U1: AP33772S, Package_DFN_QFN:QFN-24-1EP_4x4mm_P0.5mm_EP2.6x2.6mm, F.Cu at (32.0, 30.0)
- added U2: ESP32-S3-WROOM-1, RF_Module:ESP32-S3-WROOM-1, F.Cu at (75.0, 35.0)
- added U3: NCV7240, Package_SO:SSOP-24_5.3x8.2mm_P0.65mm, F.Cu at (108.0, 18.0)
- added U4: NCV7240, Package_SO:SSOP-24_5.3x8.2mm_P0.65mm, F.Cu at (108.0, 46.0)
- added U5: NCV7240, Package_SO:SSOP-24_5.3x8.2mm_P0.65mm, F.Cu at (108.0, 74.0)
- added U6: NCV7240, Package_SO:SSOP-24_5.3x8.2mm_P0.65mm, F.Cu at (108.0, 102.0)
- added U7: TPS62932, Package_TO_SOT_SMD:SOT-23-6, F.Cu at (18.0, 60.0)
- moved MH4 44.7 mm to (196.0, 116.0)
- moved MH2 40.0 mm to (196.0, 4.00)
- moved MH3 20.0 mm to (4.00, 116.0)
Routing:
- net GND: vias 0 -> 48
- added copper zone on F.Cu, net +3V3
Other:
- board size 160 x 100 mm -> 200 x 120 mm
- board text added: "4× NCV7240"
- board text added: "Buck 24V→3V3"
- board text added: "ESP32-S3"
- board text added: "Flyback diodes"
- board text added: "Screw terminals"
- board text added: "USB-C PD"
- board text added: "rev 0.2 — 2026"
- board text removed: "4× NCV7240 (U3..U6 + decoupling)"
- board text removed: "Buck 24V→3V3 (U7, L1, C3, R6/R7)"
- board text removed: "ESP32-S3 (U2, C4/C5, R1..R5)"
- board text removed: "Flyback diode field (D2..D33, B260A, K→+24V)"
- board text removed: "Screw terminals (J2..J5, 32 outputs)"
- board text removed: "USB-C PD (J1, U1, C1/C2, D1)"
- board text removed: "rev 0.1 — 2026"

Commit message: Route OUTx output paths and SPI/control bus
- 32× output traces routed on F.Cu (0.5 mm width):
    NCV pin → flyback diode anode → screw terminal pin
- Shared SPI/control bus on F.Cu (0.25 mm) in the gap between
  ESP32 and the NCV stack:
    SPI_SCK   x=96
    SPI_MOSI  x=97
    SPI_MISO  x=98
    NCV_RSTB  x=99
    NCV_FSOB  x=100
  Vertical bus tracks span all 4 NCV ICs; horizontal stubs fan
  out to each NCV's left-side pin (4,5,6,7,8).
- Per-NCV /CSB stubs (CS1..CS4 independent)
- ESP32 → bus connector stubs (rough; KiCad can tidy)
- Moved screw terminals from x=180 to x=175 for 3.5 mm clearance
  to the right-edge mounting holes

Total: 72 footprints, 313 pads, 102 tracks, 48 stitching vias,
4 filled zones. PCB now has fully placed components and the
bulk of routing — only fine-tuning and DRC cleanup left.
Parts:
- removed the D17 at (148.0, 51.5)
- added C15: 10uF/50V, Capacitor_SMD:C_1210_3225Metric, F.Cu at (120.0, 79.0)
- D17: renamed from U5; value NCV7240 -> B260A; footprint Package_SO:SSOP-24_5.3x8.2mm_P0.65mm -> Diode_SMD:D_SMA
- U5: renamed from C15; value 10uF/50V -> NCV7240; footprint Capacitor_SMD:C_1210_3225Metric -> Package_SO:SSOP-24_5.3x8.2mm_P0.65mm
- moved D17 45.9 mm to (148.0, 51.5)
- moved U5 13.0 mm to (108.0, 74.0)
- moved J2 5.00 mm to (175.0, 18.0)
- moved J3 5.00 mm to (175.0, 46.0)
- moved J4 5.00 mm to (175.0, 74.0)
- moved J5 5.00 mm to (175.0, 102.0)
Connections:
- D17 pad 2: +3V3 -> OUT16
- U5 pad 2: GND -> +3V3
Routing:
- net SPI_SCK: track 0.00 -> 148.7 mm
- net SPI_MOSI: track 0.00 -> 145.7 mm
- net SPI_MISO: track 0.00 -> 142.7 mm
- net NCV_RSTB: track 0.00 -> 139.7 mm
- net NCV_FSOB: track 0.00 -> 136.7 mm
- net OUT8: track 0.00 -> 82.4 mm
- net OUT32: track 0.00 -> 82.4 mm
- net OUT24: track 0.00 -> 82.4 mm
- net OUT16: track 0.00 -> 82.4 mm
- net OUT7: track 0.00 -> 76.6 mm
- net OUT31: track 0.00 -> 76.6 mm
- net OUT23: track 0.00 -> 76.6 mm
- net OUT15: track 0.00 -> 76.6 mm
- net OUT6: track 0.00 -> 71.7 mm
- net OUT30: track 0.00 -> 71.7 mm
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
Commit message: pcb: add F.Cu GND zone, populate fp-lib-table, render board
- Add low-priority F.Cu GND copper pour so perimeter stitching vias
  have something to anchor to on the top side.
- Populate fp-lib-table with standard KiCad footprint libraries
  (Resistor_SMD, Capacitor_SMD, Diode_SMD, Package_SO, Package_DFN_QFN,
  RF_Module, Connector_USB, TerminalBlock_Phoenix, MountingHole, etc.)
  so KiCad GUI can resolve real library footprints when the user runs
  "Update PCB from Schematic".
- Commit top/bottom render PNGs for quick review.
- Ignore *.rpt files (DRC outputs).

DRC state: 400 violations remain (219 unconnected nets needing routing,
150 solder-mask bridges from placeholder OUTx tracks, 66 lib-footprint
mismatches that will resolve after schematic-driven update, plus zones,
crossings and dangling vias). Placement is complete; routing must be
finished in the KiCad GUI.
Routing:
- added copper zone on F.Cu, net GND

Commit message: pcb: freerouting headless round-trip (partial)
Set up a headless DSN→freerouting→SES round-trip:
- DSN export via pcbnew Python bindings (ExportSpecctraDSN)
- freerouting v2.2.3 run with --gui-disabled, 30 router passes,
  5 optimizer passes, 10-minute job timeout
- SES import via pcbnew.ImportSpecctraSES

Result: partial autoroute. 137 net segments at start, 98 still
unrouted at timeout. DRC: 412 violations (196 unconnected items,
150 solder-mask bridges, 67 tracks crossing, 62 dangling vias,
plus the 66 lib_footprint_mismatch that will clear once the user
runs Update PCB from Schematic in the GUI).

Why incomplete: KiCad placement was done by gen_pcb.py using
placeholder pad geometries; pads end up slightly off the real
library footprints, so freerouting sees a less optimal board than
it would after schematic-driven update. Useful as a preview, not
as a finished route.

Artefacts committed: ncv7240-driver.dsn (input), ncv7240-driver.ses
(freerouting output), board-{top,bottom}-routed.png renders.
Routing:
- net USB_D+: track 0.00 -> 115.7 mm, vias 0 -> 2
- net EN_3V3: track 0.00 -> 81.4 mm, vias 0 -> 3
- net I2C_SCL: track 0.00 -> 71.0 mm, vias 0 -> 2
- net I2C_SDA: track 0.00 -> 64.6 mm, vias 0 -> 2
- net USB_D-: track 0.00 -> 60.8 mm
- net +3V3: track 0.00 -> 40.9 mm, vias 0 -> 4
- net SPI_CS3: track 20.5 -> 56.0 mm, vias 0 -> 2
- net PD_INT: track 0.00 -> 34.3 mm
- net +24V: track 0.00 -> 27.1 mm, vias 0 -> 13
- net VBUS: track 0.00 -> 23.4 mm
- net CC1: track 0.00 -> 22.8 mm, vias 0 -> 2
- net SPI_CS2: track 20.5 -> 37.1 mm, vias 0 -> 2
- net FB: track 0.00 -> 16.6 mm
- net SW: track 0.00 -> 14.3 mm
- net NCV_RSTB: track 139.7 -> 150.5 mm
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